File: LED_Keychain_rev2.brd (EAGLE design)
At the start: 50.8 x 50.8 mm, 6 parts

Commit message: Added functional rev2
Parts:
- LED1, LED2, LED3: value RGBLED5050 -> KINGBRIGHT-A1608; device adafruit:RGBLED5050 -> LED_Keychain_lib:KINGBRIGHT-0603
- moved LED1 1.27 mm to (12.7, 29.2), turned to 90 degrees
- moved LED2 1.27 mm to (25.4, 29.2), turned to 90 degrees
- moved LED3 1.27 mm to (38.1, 29.2), turned to 90 degrees
Connections:
- net LEDOUT: now also LED1.CATHODE, LED2.CATHODE, LED3.CATHODE; no longer LED1.5, LED2.5, LED3.5
- net VCC: now also LED1.ANODE, LED2.ANODE, LED3.ANODE; no longer LED1.2, LED2.2, LED3.2
Changed lines of the file:
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@@
 <drawing>
 <settings>
-<setting alwaysvectorfont="yes"/>
+<setting alwaysvectorfont="no"/>
 <setting verticaltext="up"/>
 </settings>
@@
 <attribute name="NAME" x="13.97" y="58.42" size="3.81" layer="26" rot="MR0"/>
 </element>
-<element name="LED1" library="adafruit" package="RGBLED5050" value="RGBLED5050" x="12.7" y="30.48" smashed="yes" rot="R270">
-<attribute name="NAME" x="10.52" y="34.72" size="1.27" layer="25" font="vector"/>
-<attribute name="VALUE" x="8.16" y="25.11" size="1.27" layer="27" font="vector"/>
-</element>
 <element name="R1" library="adafruit" package="R0603" value="" x="25.4" y="19.05" smashed="yes" rot="R270">
 <attribute name="NAME" x="26.289" y="19.939" size="1.27" layer="25" rot="R270"/>
 <attribute name="VALUE" x="23.368" y="19.939" size="1.27" layer="27" rot="R270"/>
 </element>
-<element name="LED2" library="adafruit" package="RGBLED5050" value="RGBLED5050" x="25.4" y="30.48" smashed="yes" rot="R270">
-<attribute name="NAME" x="23.22" y="34.72" size="1.27" layer="25" font="vector"/>
-<attribute name="VALUE" x="20.86" y="25.11" size="1.27" layer="27" font="vector"/>
-</element>
-<element name="LED3" library="adafruit" package="RGBLED5050" value="RGBLED5050" x="38.1" y="30.48" smashed="yes" rot="R270">
-<attribute name="NAME" x="35.92" y="34.72" size="1.27" layer="25" font="vector"/>
-<attribute name="VALUE" x="33.56" y="25.11" size="1.27" layer="27" font="vector"/>
+<element name="LED1" library="LED_Keychain_lib" package="KINGBRIGHT-0603" value="KINGBRIGHT-A1608" x="12.7" y="29.21" smashed="yes" rot="R90">
+<attribute name="NAME" x="14.7" y="32.02" size="1.27" layer="25" rot="R180"/>
+</element>
+<element name="LED2" library="LED_Keychain_lib" package="KINGBRIGHT-0603" value="KINGBRIGHT-A1608" x="25.4" y="29.21" smashed="yes" rot="R90">
+<attribute name="NAME" x="27.4" y="32.02" size="1.27" layer="25" rot="R180"/>
+</element>
+<element name="LED3" library="LED_Keychain_lib" package="KINGBRIGHT-0603" value="KINGBRIGHT-A1608" x="38.1" y="29.21" smashed="yes" rot="R90">
+<attribute name="NAME" x="40.1" y="32.02" size="1.27" layer="25" rot="R180"/>
 </element>
 </elements>
@@
 <contactref element="U$1" pad="VCC1"/>
 <contactref element="U$1" pad="VCC2"/>
-<contactref element="LED1" pad="2"/>
-<contactref element="LED2" pad="2"/>
-<contactref element="LED3" pad="2"/>
 <polygon width="0.1524" layer="1">
 <vertex x="-21.59" y="48.26"/>
@@
 <vertex x="15.24" y="85.09"/>
 </polygon>
+<contactref element="LED1" pad="ANODE"/>
+<contactref element="LED2" pad="ANODE"/>
+<contactref element="LED3" pad="ANODE"/>
 </signal>
 <signal name="LEDOUT">
 <contactref element="R1" pad="1"/>
-<contactref element="LED1" pad="5"/>
-<contactref element="LED2" pad="5"/>
-<contactref element="LED3" pad="5"/>
-<wire x1="12.7" y1="28.48" x2="12.7" y2="26.67" width="0.4064" layer="1"/>
 <wire x1="12.7" y1="26.67" x2="15.24" y2="24.13" width="0.4064" layer="1"/>
 <wire x1="15.24" y1="24.13" x2="24.13" y2="24.13" width="0.4064" layer="1"/>
 <wire x1="24.13" y1="24.13" x2="25.4" y2="22.86" width="0.4064" layer="1"/>
 <wire x1="25.4" y1="22.86" x2="25.4" y2="19.9" width="0.4064" layer="1"/>
-<wire x1="38.1" y1="28.48" x2="38.1" y2="26.67" width="0.4064" layer="1"/>
 <wire x1="38.1" y1="26.67" x2="35.56" y2="24.13" width="0.4064" layer="1"/>
 <wire x1="35.56" y1="24.13" x2="26.67" y2="24.13" width="0.4064" layer="1"/>
 <wire x1="26.67" y1="24.13" x2="25.4" y2="22.86" width="0.4064" layer="1"/>
-<wire x1="25.4" y1="28.48" x2="25.4" y2="22.86" width="0.4064" layer="1"/>
+<contactref element="LED1" pad="CATHODE"/>
+<contactref element="LED2" pad="CATHODE"/>
+<contactref element="LED3" pad="CATHODE"/>
+<wire x1="12.7" y1="28.565" x2="12.7" y2="26.67" width="0.4064" layer="1"/>
+<wire x1="25.4" y1="28.565" x2="25.4" y2="22.86" width="0.4064" layer="1"/>
+<wire x1="38.1" y1="28.565" x2="38.1" y2="26.67" width="0.4064" layer="1"/>
 </signal>
 </signals>
