File: LED_Keychain_rev2.sch (EAGLE design)
At the start: 6 parts

Commit message: Added functional rev2
Parts:
- LED1, LED2, LED3: value RGBLED5050 -> KINGBRIGHT-A1608; device adafruit:RGBLED5050 -> LED_Keychain_lib:KINGBRIGHT-A1608
Connections:
- net LEDOUT: now also LED1.CATHODE, LED2.CATHODE, LED3.CATHODE; no longer LED1.RED_C, LED2.RED_C, LED3.RED_C
- net VCC: now also LED1.ANODE, LED2.ANODE, LED3.ANODE; no longer LED1.RED_A, LED2.RED_A, LED3.RED_A
Changed lines of the file:
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@@
 <part name="U$2" library="Keyboard" deviceset="KEYSWITCH-PLAIN" device="-MX-1U"/>
 <part name="U$1" library="LED_Keychain_lib" deviceset="KEYSTONE3035" device=""/>
-<part name="LED1" library="adafruit" deviceset="RGBLED" device="5050"/>
 <part name="R1" library="adafruit" deviceset="R-US_" device="R0603"/>
 <part name="GND1" library="supply1" library_urn="urn:adsk.eagle:library:371" deviceset="GND" device=""/>
 <part name="P+1" library="supply1" library_urn="urn:adsk.eagle:library:371" deviceset="VCC" device=""/>
-<part name="LED2" library="adafruit" deviceset="RGBLED" device="5050"/>
-<part name="LED3" library="adafruit" deviceset="RGBLED" device="5050"/>
+<part name="LED1" library="LED_Keychain_lib" deviceset="KINGBRIGHT-A1608" device=""/>
+<part name="LED2" library="LED_Keychain_lib" deviceset="KINGBRIGHT-A1608" device=""/>
+<part name="LED3" library="LED_Keychain_lib" deviceset="KINGBRIGHT-A1608" device=""/>
 </parts>
 <sheets>
@@
 <attribute name="NAME" x="213.36" y="93.98" size="1.778" layer="95"/>
 </instance>
-<instance part="LED1" gate="G$1" x="190.5" y="50.8" smashed="yes">
-<attribute name="NAME" x="186.69" y="59.69" size="1.778" layer="95"/>
-</instance>
 <instance part="R1" gate="G$1" x="246.38" y="96.52" smashed="yes">
 <attribute name="NAME" x="242.57" y="98.0186" size="1.778" layer="95"/>
@@
 <attribute name="VALUE" x="200.66" y="101.6" size="1.778" layer="96" rot="R90"/>
 </instance>
-<instance part="LED2" gate="G$1" x="220.98" y="50.8" smashed="yes">
-<attribute name="NAME" x="217.17" y="59.69" size="1.778" layer="95"/>
+<instance part="LED1" gate="G$1" x="187.96" y="45.72" smashed="yes" rot="R90">
+<attribute name="NAME" x="192.532" y="49.276" size="1.778" layer="95" rot="R180"/>
 </instance>
-<instance part="LED3" gate="G$1" x="251.46" y="50.8" smashed="yes">
-<attribute name="NAME" x="247.65" y="59.69" size="1.778" layer="95"/>
+<instance part="LED2" gate="G$1" x="218.44" y="45.72" smashed="yes" rot="R90">
+<attribute name="NAME" x="223.012" y="49.276" size="1.778" layer="95" rot="R180"/>
+</instance>
+<instance part="LED3" gate="G$1" x="248.92" y="45.72" smashed="yes" rot="R90">
+<attribute name="NAME" x="253.492" y="49.276" size="1.778" layer="95" rot="R180"/>
 </instance>
 </instances>
@@
 </segment>
 <segment>
-<pinref part="LED1" gate="G$1" pin="RED_A"/>
 <wire x1="185.42" y1="45.72" x2="177.8" y2="45.72" width="0.1524" layer="91"/>
 <label x="177.8" y="43.18" size="1.778" layer="95"/>
+<pinref part="LED1" gate="G$1" pin="ANODE"/>
 </segment>
 <segment>
-<pinref part="LED2" gate="G$1" pin="RED_A"/>
 <wire x1="215.9" y1="45.72" x2="208.28" y2="45.72" width="0.1524" layer="91"/>
 <label x="208.28" y="43.18" size="1.778" layer="95"/>
+<pinref part="LED2" gate="G$1" pin="ANODE"/>
 </segment>
 <segment>
-<pinref part="LED3" gate="G$1" pin="RED_A"/>
 <wire x1="246.38" y1="45.72" x2="238.76" y2="45.72" width="0.1524" layer="91"/>
 <label x="238.76" y="43.18" size="1.778" layer="95"/>
+<pinref part="LED3" gate="G$1" pin="ANODE"/>
 </segment>
 </net>
@@
 </segment>
 <segment>
-<pinref part="LED1" gate="G$1" pin="RED_C"/>
-<wire x1="195.58" y1="45.72" x2="203.2" y2="45.72" width="0.1524" layer="91"/>
+<wire x1="193.04" y1="45.72" x2="203.2" y2="45.72" width="0.1524" layer="91"/>
 <label x="195.58" y="43.18" size="1.778" layer="95"/>
+<pinref part="LED1" gate="G$1" pin="CATHODE"/>
 </segment>
 <segment>
-<pinref part="LED2" gate="G$1" pin="RED_C"/>
-<wire x1="226.06" y1="45.72" x2="233.68" y2="45.72" width="0.1524" layer="91"/>
+<wire x1="223.52" y1="45.72" x2="233.68" y2="45.72" width="0.1524" layer="91"/>
 <label x="226.06" y="43.18" size="1.778" layer="95"/>
+<pinref part="LED2" gate="G$1" pin="CATHODE"/>
 </segment>
 <segment>
-<pinref part="LED3" gate="G$1" pin="RED_C"/>
-<wire x1="256.54" y1="45.72" x2="264.16" y2="45.72" width="0.1524" layer="91"/>
+<wire x1="254" y1="45.72" x2="264.16" y2="45.72" width="0.1524" layer="91"/>
 <label x="256.54" y="43.18" size="1.778" layer="95"/>
+<pinref part="LED3" gate="G$1" pin="CATHODE"/>
 </segment>
 </net>
